Commit message: add muse state estimator

File: tbai_ros_description/urdf/anymal_d_gazebo_blind.urdf.xacro (robot description, xacro)
@@ -30,12 +30,12 @@
 <!-- State publisher -->
 <gazebo>
-  <plugin filename="/home/kuba/Documents/ros/devel/.private/tbai_ros_gazebo/lib/libStatePublisher.so" name="StatePublisher"/>
+  <plugin filename="/home/kuba/Documents/ros/devel/.private/tbai_ros_gazebo/lib/libRobotStatePublisher.so" name="RobotStatePublisher"/>
 </gazebo>
 <!-- Add contact sensors -->
 <gazebo reference="LF_FOOT">
     <sensor name="lf_foot_contact" type="contact">
-    <plugin name="lf_contact_plugin" filename="libContactSensor.so"/>
+    <plugin name="lf_contact_plugin" filename="/home/kuba/Documents/ros/devel/.private/tbai_ros_gazebo/lib/libContactSensor.so"/>
     <contact>
-        <collision>LF_SHANK_fixed_joint_lump__LF_FOOT_collision_3</collision>
+        <collision>LF_SHANK_fixed_joint_lump__LF_FOOT_collision_sensor_collision_3</collision>
     </contact>
     </sensor>
@@ -43,7 +43,7 @@
 <gazebo reference="RF_FOOT">
     <sensor name="rf_foot_contact" type="contact">
-    <plugin name="rf_contact_plugin" filename="libContactSensor.so"/>
+    <plugin name="rf_contact_plugin" filename="/home/kuba/Documents/ros/devel/.private/tbai_ros_gazebo/lib/libContactSensor.so"/>
     <contact>
-        <collision>RF_SHANK_fixed_joint_lump__RF_FOOT_collision_3</collision>
+        <collision>RF_SHANK_fixed_joint_lump__RF_FOOT_collision_sensor_collision_3</collision>
     </contact>
     </sensor>
@@ -51,7 +51,7 @@
 <gazebo reference="LH_FOOT">
     <sensor name="lh_foot_contact" type="contact">
-    <plugin name="lh_contact_plugin" filename="libContactSensor.so"/>
+    <plugin name="lh_contact_plugin" filename="/home/kuba/Documents/ros/devel/.private/tbai_ros_gazebo/lib/libContactSensor.so"/>
     <contact>
-        <collision>LH_SHANK_fixed_joint_lump__LH_FOOT_collision_3</collision>
+        <collision>LH_SHANK_fixed_joint_lump__LH_FOOT_collision_sensor_collision_3</collision>
     </contact>
     </sensor>
@@ -59,7 +59,7 @@
 <gazebo reference="RH_FOOT">
     <sensor name="rh_foot_contact" type="contact">
-    <plugin name="rh_contact_plugin" filename="libContactSensor.so"/>
+    <plugin name="rh_contact_plugin" filename="/home/kuba/Documents/ros/devel/.private/tbai_ros_gazebo/lib/libContactSensor.so"/>
     <contact>
-        <collision>RH_SHANK_fixed_joint_lump__RH_FOOT_collision_3</collision>
+        <collision>RH_SHANK_fixed_joint_lump__RH_FOOT_collision_sensor_collision_3</collision>
     </contact>
     </sensor>
