Commit message: updates for go2

File: tbai_ros_description/urdf/anymal_d_gazebo_blind.urdf.xacro (robot description, xacro)
@@ -37,5 +37,5 @@
     <plugin name="lf_contact_plugin" filename="/home/kuba/Documents/ros/devel/.private/tbai_ros_gazebo/lib/libContactSensor.so"/>
     <contact>
-        <collision>LF_SHANK_fixed_joint_lump__LF_FOOT_collision_sensor_collision_3</collision>
+        <collision>FL_calf_fixed_joint_lump__LF_FOOT_collision_sensor_collision_3</collision>
     </contact>
     </sensor>
@@ -45,5 +45,5 @@
     <plugin name="rf_contact_plugin" filename="/home/kuba/Documents/ros/devel/.private/tbai_ros_gazebo/lib/libContactSensor.so"/>
     <contact>
-        <collision>RF_SHANK_fixed_joint_lump__RF_FOOT_collision_sensor_collision_3</collision>
+        <collision>FR_calf_fixed_joint_lump__RF_FOOT_collision_sensor_collision_3</collision>
     </contact>
     </sensor>
@@ -53,5 +53,5 @@
     <plugin name="lh_contact_plugin" filename="/home/kuba/Documents/ros/devel/.private/tbai_ros_gazebo/lib/libContactSensor.so"/>
     <contact>
-        <collision>LH_SHANK_fixed_joint_lump__LH_FOOT_collision_sensor_collision_3</collision>
+        <collision>RL_calf_fixed_joint_lump__LH_FOOT_collision_sensor_collision_1</collision>
     </contact>
     </sensor>
@@ -61,5 +61,5 @@
     <plugin name="rh_contact_plugin" filename="/home/kuba/Documents/ros/devel/.private/tbai_ros_gazebo/lib/libContactSensor.so"/>
     <contact>
-        <collision>RH_SHANK_fixed_joint_lump__RH_FOOT_collision_sensor_collision_3</collision>
+        <collision>RR_calf_fixed_joint_lump__RH_FOOT_collision_sensor_collision_1</collision>
     </contact>
     </sensor>

File: tbai_ros_description/urdf/go2_gazebo_blind.urdf.xacro (robot description, xacro)
@@ -30,5 +30,38 @@
 <!-- State publisher -->
 <gazebo>
-  <plugin filename="/home/kuba/Documents/ros/devel/.private/tbai_ros_gazebo/lib/libStatePublisher.so" name="StatePublisher"/>
+  <plugin filename="/home/kuba/Documents/ros/devel/.private/tbai_ros_gazebo/lib/libRobotStatePublisher.so" name="RobotStatePublisher"/>
+</gazebo>
+<!-- Add contact sensors -->
+<gazebo reference="LF_FOOT">
+    <sensor name="lf_foot_contact" type="contact">
+    <plugin name="lf_contact_plugin" filename="/home/kuba/Documents/ros/devel/.private/tbai_ros_gazebo/lib/libContactSensor.so"/>
+    <contact>
+        <collision>FL_calf_fixed_joint_lump__LF_FOOT_collision_sensor_collision_3</collision>
+    </contact>
+    </sensor>
+</gazebo>
+<gazebo reference="RF_FOOT">
+    <sensor name="rf_foot_contact" type="contact">
+    <plugin name="rf_contact_plugin" filename="/home/kuba/Documents/ros/devel/.private/tbai_ros_gazebo/lib/libContactSensor.so"/>
+    <contact>
+        <collision>FR_calf_fixed_joint_lump__RF_FOOT_collision_sensor_collision_3</collision>
+    </contact>
+    </sensor>
+</gazebo>
+<gazebo reference="LH_FOOT">
+    <sensor name="lh_foot_contact" type="contact">
+    <plugin name="lh_contact_plugin" filename="/home/kuba/Documents/ros/devel/.private/tbai_ros_gazebo/lib/libContactSensor.so"/>
+    <contact>
+        <collision>RL_calf_fixed_joint_lump__LH_FOOT_collision_sensor_collision_1</collision>
+    </contact>
+    </sensor>
+</gazebo>
+<gazebo reference="RH_FOOT">
+    <sensor name="rh_foot_contact" type="contact">
+    <plugin name="rh_contact_plugin" filename="/home/kuba/Documents/ros/devel/.private/tbai_ros_gazebo/lib/libContactSensor.so"/>
+    <contact>
+        <collision>RR_calf_fixed_joint_lump__RH_FOOT_collision_sensor_collision_1</collision>
+    </contact>
+    </sensor>
 </gazebo>
 <!-- Gazebo materials -->

File: tbai_ros_description/urdf/model.urdf (robot description, URDF)
Before this commit: robot anymal_d, 87 links, 86 joints
Links:
- removed link LF_HAA_drive
- removed link LF_HFE_drive
- removed link LF_HFE_output
- removed link LF_HIP
- removed link LF_KFE_drive
- removed link LF_SHANK
- removed link LF_THIGH
- removed link LF_hip_fixed
- removed link LF_shank_fixed
- removed link LF_thigh_fixed
- removed link LH_HAA_drive
- removed link LH_HFE_drive
- removed link LH_HFE_output
- removed link LH_HIP
- removed link LH_KFE_drive
- removed link LH_SHANK
- removed link LH_THIGH
- removed link LH_hip_fixed
- removed link LH_shank_fixed
- removed link LH_thigh_fixed
- removed link RF_HAA_drive
- removed link RF_HFE_drive
- removed link RF_HFE_output
- removed link RF_HIP
- removed link RF_KFE_drive
- removed link RF_SHANK
- removed link RF_THIGH
- removed link RF_hip_fixed
- removed link RF_shank_fixed
- removed link RF_thigh_fixed
- removed link RH_HAA_drive
- removed link RH_HFE_drive
- removed link RH_HFE_output
- removed link RH_HIP
- removed link RH_KFE_drive
- removed link RH_SHANK
- removed link RH_THIGH
- removed link RH_hip_fixed
- removed link RH_shank_fixed
- removed link RH_thigh_fixed
- removed link base_inertia
- removed link battery
- removed link body_top
- removed link bottom_shell
- removed link depth_camera_front_lower_camera
- removed link depth_camera_front_lower_camera_parent
- removed link depth_camera_front_lower_depth_frame
- removed link depth_camera_front_lower_depth_optical_frame
- removed link depth_camera_front_upper_camera
- removed link depth_camera_front_upper_camera_parent
- removed link depth_camera_front_upper_depth_frame
- removed link depth_camera_front_upper_depth_optical_frame
- removed link depth_camera_left_camera
- removed link depth_camera_left_camera_parent
- removed link depth_camera_left_depth_frame
- removed link depth_camera_left_depth_optical_frame
- removed link depth_camera_rear_lower_camera
- removed link depth_camera_rear_lower_camera_parent
- removed link depth_camera_rear_lower_depth_frame
- removed link depth_camera_rear_lower_depth_optical_frame
- removed link depth_camera_rear_upper_camera
- removed link depth_camera_rear_upper_camera_parent
- removed link depth_camera_rear_upper_depth_frame
- removed link depth_camera_rear_upper_depth_optical_frame
- removed link depth_camera_right_camera
- removed link depth_camera_right_camera_parent
- removed link depth_camera_right_depth_frame
- removed link depth_camera_right_depth_optical_frame
- removed link docking_socket
- removed link face_front
- removed link face_rear
- removed link face_shell_front
- removed link face_shell_rear
- removed link hbc_receiver
- removed link imu_link
- removed link lidar
- removed link lidar_parent
- removed link top_shell
- removed link wide_angle_camera_front_camera
- removed link wide_angle_camera_front_camera_parent
- removed link wide_angle_camera_rear_camera
- removed link wide_angle_camera_rear_camera_parent
- added link FL_calf, mass 0.154; collision cylinder length=0.12 radius=0.012; visual mesh filename=package://ocs2_robotic_assets/resources/go2/dae/calf.dae
- added link FL_calf_rotor, mass 0.089
- added link FL_calflower; collision cylinder length=0.065 radius=0.011
- added link FL_calflower1; collision cylinder length=0.03 radius=0.0155
- added link FL_hip, mass 0.678; collision cylinder length=0.04 radius=0.046; visual mesh filename=package://ocs2_robotic_assets/resources/go2/dae/hip.dae
- added link FL_hip_rotor, mass 0.089
- added link FL_thigh, mass 1.152; collision box size=0.213 0.0245 0.034; visual mesh filename=package://ocs2_robotic_assets/resources/go2/dae/thigh.dae
- added link FL_thigh_rotor, mass 0.089
- added link FR_calf, mass 0.154; collision cylinder length=0.12 radius=0.013; visual mesh filename=package://ocs2_robotic_assets/resources/go2/dae/calf_mirror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
- added link FR_calf_rotor, mass 0.089
- added link FR_calflower; collision cylinder length=0.065 radius=0.011
- added link FR_calflower1; collision cylinder length=0.03 radius=0.0155
- added link FR_hip, mass 0.678; collision cylinder length=0.04 radius=0.046; visual mesh filename=package://ocs2_robotic_assets/resources/go2/dae/hip.dae
- added link FR_hip_rotor, mass 0.089
- added link FR_thigh, mass 1.152; collision box size=0.213 0.0245 0.034; visual mesh filename=package://ocs2_robotic_assets/resources/go2/dae/thigh_mirro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
- added link FR_thigh_rotor, mass 0.089
- added link Head_lower, mass 0.001; collision sphere radius=0.047
- added link Head_upper, mass 0.001; collision cylinder length=0.09 radius=0.05
- added link RL_calf, mass 0.154; collision cylinder length=0.12 radius=0.013; visual mesh filename=package://ocs2_robotic_assets/resources/go2/dae/calf.dae
- added link RL_calf_rotor, mass 0.089
- added link RL_calflower; collision cylinder length=0.065 radius=0.011
- added link RL_calflower1; collision cylinder length=0.03 radius=0.0155
- added link RL_hip, mass 0.678; collision cylinder length=0.04 radius=0.046; visual mesh filename=package://ocs2_robotic_assets/resources/go2/dae/hip.dae
- added link RL_hip_rotor, mass 0.089
- added link RL_thigh, mass 1.152; collision box size=0.213 0.0245 0.034; visual mesh filename=package://ocs2_robotic_assets/resources/go2/dae/thigh.dae
- added link RL_thigh_rotor, mass 0.089
- added link RR_calf, mass 0.154; collision cylinder length=0.12 radius=0.013; visual mesh filename=package://ocs2_robotic_assets/resources/go2/dae/calf_mirror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
- added link RR_calf_rotor, mass 0.089
- added link RR_calflower; collision cylinder length=0.065 radius=0.011
- added link RR_calflower1; collision cylinder length=0.03 radius=0.0155
- added link RR_hip, mass 0.678; collision cylinder length=0.04 radius=0.046; visual mesh filename=package://ocs2_robotic_assets/resources/go2/dae/hip.dae
- added link RR_hip_rotor, mass 0.089
- added link RR_thigh, mass 1.152; collision box size=0.213 0.0245 0.034; visual mesh filename=package://ocs2_robotic_assets/resources/go2/dae/thigh_mirro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
- added link RR_thigh_rotor, mass 0.089
- added link front_camera
- added link imu, mass 0
- added link radar, mass 0
- link LF_FOOT: mass 0.29644 -> 0.04; geometry collision sphere radius=0.022; visual mesh filename=package://ocs2_robotic_assets/resources/go2/dae/foot.dae
- link LH_FOOT: mass 0.29644 -> 0.04; geometry collision sphere radius=0.022; visual mesh filename=package://ocs2_robotic_assets/resources/go2/dae/foot.dae
- link RF_FOOT: mass 0.29644 -> 0.04; geometry collision sphere radius=0.022; visual mesh filename=package://ocs2_robotic_assets/resources/go2/dae/foot.dae
- link RH_FOOT: mass 0.29644 -> 0.04; geometry collision sphere radius=0.022; visual mesh filename=package://ocs2_robotic_assets/resources/go2/dae/foot.dae
- link base: mass None -> 6.921; geometry collision box size=0.3762 0.0935 0.114; visual mesh filename=package://ocs2_robotic_assets/resources/go2/dae/base.dae
Joints:
- removed joint LF_HFE_drive_LF_thigh_fixed
- removed joint LF_HIP_LF_hip_fixed
- removed joint LF_THIGH_to_LF_HFE_drive
- removed joint LF_hip_fixed_LF_HFE_output
- removed joint LF_shank_LF_shank_fixed
- removed joint LF_shank_fixed_LF_FOOT
- removed joint LF_thigh_fixed_LF_KFE_drive
- removed joint LH_HFE_drive_LH_thigh_fixed
- removed joint LH_HIP_LH_hip_fixed
- removed joint LH_THIGH_to_LH_HFE_drive
- removed joint LH_hip_fixed_LH_HFE_output
- removed joint LH_shank_LH_shank_fixed
- removed joint LH_shank_fixed_LH_FOOT
- removed joint LH_thigh_fixed_LH_KFE_drive
- removed joint RF_HFE_drive_RF_thigh_fixed
- removed joint RF_HIP_RF_hip_fixed
- removed joint RF_THIGH_to_RF_HFE_drive
- removed joint RF_hip_fixed_RF_HFE_output
- removed joint RF_shank_RF_shank_fixed
- removed joint RF_shank_fixed_RF_FOOT
- removed joint RF_thigh_fixed_RF_KFE_drive
- removed joint RH_HFE_drive_RH_thigh_fixed
- removed joint RH_HIP_RH_hip_fixed
- removed joint RH_THIGH_to_RH_HFE_drive
- removed joint RH_hip_fixed_RH_HFE_output
- removed joint RH_shank_RH_shank_fixed
- removed joint RH_shank_fixed_RH_FOOT
- removed joint RH_thigh_fixed_RH_KFE_drive
- removed joint base_LF_HAA_drive
- removed joint base_LH_HAA_drive
- removed joint base_RF_HAA_drive
- removed joint base_RH_HAA_drive
- removed joint base_battery
- removed joint base_bottom_shell
- removed joint base_face_front
- removed joint base_face_rear
- removed joint base_face_shell_front
- removed joint base_face_shell_rear
- removed joint base_hbc_receiver
- removed joint base_to_base_inertia
- removed joint base_to_body_top
- removed joint base_to_depth_camera_left_camera
- removed joint base_to_depth_camera_right_camera
- removed joint base_to_docking_socket
- removed joint base_to_lidar_parent
- removed joint base_top_shell
- removed joint depth_camera_front_lower_camera_depth_to_depth_optical_frame
- removed joint depth_camera_front_lower_camera_parent_to_depth_frame
- removed joint depth_camera_front_lower_camera_to_camera_parent
- removed joint depth_camera_front_upper_camera_depth_to_depth_optical_frame
- removed joint depth_camera_front_upper_camera_parent_to_depth_frame
- removed joint depth_camera_front_upper_camera_to_camera_parent
- removed joint depth_camera_left_camera_depth_to_depth_optical_frame
- removed joint depth_camera_left_camera_parent_to_depth_frame
- removed joint depth_camera_left_camera_to_camera_parent
- removed joint depth_camera_rear_lower_camera_depth_to_depth_optical_frame
- removed joint depth_camera_rear_lower_camera_parent_to_depth_frame
- removed joint depth_camera_rear_lower_camera_to_camera_parent
- removed joint depth_camera_rear_upper_camera_depth_to_depth_optical_frame
- removed joint depth_camera_rear_upper_camera_parent_to_depth_frame
- removed joint depth_camera_rear_upper_camera_to_camera_parent
- removed joint depth_camera_right_camera_depth_to_depth_optical_frame
- removed joint depth_camera_right_camera_parent_to_depth_frame
- removed joint depth_camera_right_camera_to_camera_parent
- removed joint face_front_to_depth_camera_front_lower_camera
- removed joint face_front_to_depth_camera_front_upper_camera
- removed joint face_front_to_wide_angle_camera_front_camera
- removed joint face_rear_to_depth_camera_rear_lower_camera
- removed joint face_rear_to_depth_camera_rear_upper_camera
- removed joint face_rear_to_wide_angle_camera_rear_camera
- removed joint lidar_parent_to_lidar
- removed joint wide_angle_camera_front_camera_to_camera_parent
- removed joint wide_angle_camera_rear_camera_to_camera_parent
- added joint FL_calf_rotor_joint: type fixed, parent FL_thigh, child FL_calf_rotor, origin xyz=0 -0.03235 0 rpy=0 0 0
- added joint FL_calflower1_joint: type fixed, parent FL_calflower, child FL_calflower1, origin xyz=-0.01 0 -0.04 rpy=0 0.48 0, axis 0 0 0
- added joint FL_calflower_joint: type fixed, parent FL_calf, child FL_calflower, origin xyz=0.020 0 -0.148 rpy=0 0.05 0, axis 0 0 0
- added joint FL_hip_rotor_joint: type fixed, parent base, child FL_hip_rotor, origin xyz=0.11215 0.04675 0 rpy=0 0 0
- added joint FL_thigh_rotor_joint: type fixed, parent FL_hip, child FL_thigh_rotor, origin xyz=0 -0.00015 0 rpy=0 0 0
- added joint FR_calf_rotor_joint: type fixed, parent FR_thigh, child FR_calf_rotor, origin xyz=0 0.03235 0 rpy=0 0 0
- added joint FR_calflower1_joint: type fixed, parent FR_calflower, child FR_calflower1, origin xyz=-0.01 0 -0.04 rpy=0 0.48 0, axis 0 0 0
- added joint FR_calflower_joint: type fixed, parent FR_calf, child FR_calflower, origin xyz=0.020 0 -0.148 rpy=0 0.05 0, axis 0 0 0
- added joint FR_hip_rotor_joint: type fixed, parent base, child FR_hip_rotor, origin xyz=0.11215 -0.04675 0 rpy=0 0 0
- added joint FR_thigh_rotor_joint: type fixed, parent FR_hip, child FR_thigh_rotor, origin xyz=0 0.00015 0 rpy=0 0 0
- added joint Head_lower_joint: type fixed, parent Head_upper, child Head_lower, origin xyz=0.008 0 -0.07 rpy=0 0 0, axis 0 0 0
- added joint Head_upper_joint: type fixed, parent base, child Head_upper, origin xyz=0.285 0 0.01 rpy=0 0 0, axis 0 0 0
- added joint LF_FOOT_joint: type fixed, parent FL_calf, child LF_FOOT, origin xyz=0 0 -0.213 rpy=0 0 0, axis 0 0 0
- added joint LH_FOOT_joint: type fixed, parent RL_calf, child LH_FOOT, origin xyz=0 0 -0.213 rpy=0 0 0, axis 0 0 0
- added joint RF_FOOT_joint: type fixed, parent FR_calf, child RF_FOOT, origin xyz=0 0 -0.213 rpy=0 0 0, axis 0 0 0
- added joint RH_FOOT_joint: type fixed, parent RR_calf, child RH_FOOT, origin xyz=0 0 -0.213 rpy=0 0 0, axis 0 0 0
- added joint RL_calf_rotor_joint: type fixed, parent RL_thigh, child RL_calf_rotor, origin xyz=0 -0.03235 0 rpy=0 0 0
- added joint RL_calflower1_joint: type fixed, parent RL_calflower, child RL_calflower1, origin xyz=-0.01 0 -0.04 rpy=0 0.48 0, axis 0 0 0
- added joint RL_calflower_joint: type fixed, parent RL_calf, child RL_calflower, origin xyz=0.020 0 -0.148 rpy=0 0.05 0, axis 0 0 0
- added joint RL_hip_rotor_joint: type fixed, parent base, child RL_hip_rotor, origin xyz=-0.11215 0.04675 0 rpy=0 0 0
- added joint RL_thigh_rotor_joint: type fixed, parent RL_hip, child RL_thigh_rotor, origin xyz=0 -0.00015 0 rpy=0 0 0
- added joint RR_calf_rotor_joint: type fixed, parent RR_thigh, child RR_calf_rotor, origin xyz=0 0.03235 0 rpy=0 0 0
- added joint RR_calflower1_joint: type fixed, parent RR_calflower, child RR_calflower1, origin xyz=-0.01 0 -0.04 rpy=0 0.48 0, axis 0 0 0
- added joint RR_calflower_joint: type fixed, parent RR_calf, child RR_calflower, origin xyz=0.020 0 -0.148 rpy=0 0.05 0, axis 0 0 0
- added joint RR_hip_rotor_joint: type fixed, parent base, child RR_hip_rotor, origin xyz=-0.11215 -0.04675 0 rpy=0 0 0
- added joint RR_thigh_rotor_joint: type fixed, parent RR_hip, child RR_thigh_rotor, origin xyz=0 0.00015 0 rpy=0 0 0
- added joint front_camera_joint: type fixed, parent base, child front_camera, origin xyz=0.32715 -0.00003 0.04297 rpy=0 0 0
- added joint radar_joint: type fixed, parent base, child radar, origin xyz=0.28945 0 -0.046825 rpy=0 2.8782 0, axis 0 0 0
- joint LF_HAA: child LF_HIP -> FL_hip; limit lower=-0.7853985 upper=0.6108655 effort=80.0 velocity=8.5 -> lower=-1.0472 upper=1.0472 effort=23.7 velocity=30.1; origin xyz=0 0 0 rpy=0 0 0 -> xyz=0.1934 0.0465 0 rpy=0 0 0; parent LF_HAA_drive -> base
- joint LF_HFE: axis -1 0 0 -> 0 1 0; child LF_THIGH -> FL_thigh; limit lower=-9.42477796076938 upper=9.42477796076938 effort=80.0 velocity=8.5 -> lower=-1.5708 upper=3.4907 effort=23.7 velocity=30.1; origin xyz=0 0 0 rpy=0 0 0 -> xyz=0 0.0955 0 rpy=0 0 0; parent LF_HFE_output -> FL_hip
- joint LF_KFE: axis 1 0 0 -> 0 1 0; child LF_SHANK -> FL_calf; limit lower=-9.42477796076938 upper=9.42477796076938 effort=80.0 velocity=8.5 -> lower=-2.7227 upper=-0.83776 effort=45.43 velocity=15.70; origin xyz=0 0 0 rpy=0 0 0 -> xyz=0 0 -0.213 rpy=0 0 0; parent LF_KFE_drive -> FL_thigh
- joint LH_HAA: axis -1 0 0 -> 1 0 0; child LH_HIP -> RL_hip; limit lower=-0.7853985 upper=0.6108655 effort=80.0 velocity=8.5 -> lower=-1.0472 upper=1.0472 effort=23.7 velocity=30.1; origin xyz=0 0 0 rpy=0 0 0 -> xyz=-0.1934 0.0465 0 rpy=0 0 0; parent LH_HAA_drive -> base
- joint LH_HFE: axis -1 0 0 -> 0 1 0; child LH_THIGH -> RL_thigh; limit lower=-9.42477796076938 upper=9.42477796076938 effort=80.0 velocity=8.5 -> lower=-0.5236 upper=4.5379 effort=23.7 velocity=30.1; origin xyz=0 0 0 rpy=0 0 0 -> xyz=0 0.0955 0 rpy=0 0 0; parent LH_HFE_output -> RL_hip
- joint LH_KFE: axis 1 0 0 -> 0 1 0; child LH_SHANK -> RL_calf; limit lower=-9.42477796076938 upper=9.42477796076938 effort=80.0 velocity=8.5 -> lower=-2.7227 upper=-0.83776 effort=45.43 velocity=15.70; origin xyz=0 0 0 rpy=0 0 0 -> xyz=0 0 -0.213 rpy=0 0 0; parent LH_KFE_drive -> RL_thigh
- joint RF_HAA: child RF_HIP -> FR_hip; limit lower=-0.6108655 upper=0.7853985 effort=80.0 velocity=8.5 -> lower=-1.0472 upper=1.0472 effort=23.7 velocity=30.1; origin xyz=0 0 0 rpy=0 0 0 -> xyz=0.1934 -0.0465 0 rpy=0 0 0; parent RF_HAA_drive -> base
- joint RF_HFE: axis 1 0 0 -> 0 1 0; child RF_THIGH -> FR_thigh; limit lower=-9.42477796076938 upper=9.42477796076938 effort=80.0 velocity=8.5 -> lower=-1.5708 upper=3.4907 effort=23.7 velocity=30.1; origin xyz=0 0 0 rpy=0 0 0 -> xyz=0 -0.0955 0 rpy=0 0 0; parent RF_HFE_output -> FR_hip
- joint RF_KFE: axis -1 0 0 -> 0 1 0; child RF_SHANK -> FR_calf; limit lower=-9.42477796076938 upper=9.42477796076938 effort=80.0 velocity=8.5 -> lower=-2.7227 upper=-0.83776 effort=45.43 velocity=15.70; origin xyz=0 0 0 rpy=0 0 0 -> xyz=0 0 -0.213 rpy=0 0 0; parent RF_KFE_drive -> FR_thigh
- joint RH_HAA: axis -1 0 0 -> 1 0 0; child RH_HIP -> RR_hip; limit lower=-0.6108655 upper=0.7853985 effort=80.0 velocity=8.5 -> lower=-1.0472 upper=1.0472 effort=23.7 velocity=30.1; origin xyz=0 0 0 rpy=0 0 0 -> xyz=-0.1934 -0.0465 0 rpy=0 0 0; parent RH_HAA_drive -> base
- joint RH_HFE: axis 1 0 0 -> 0 1 0; child RH_THIGH -> RR_thigh; limit lower=-9.42477796076938 upper=9.42477796076938 effort=80.0 velocity=8.5 -> lower=-0.5236 upper=4.5379 effort=23.7 velocity=30.1; origin xyz=0 0 0 rpy=0 0 0 -> xyz=0 -0.0955 0 rpy=0 0 0; parent RH_HFE_output -> RR_hip
- joint RH_KFE: axis -1 0 0 -> 0 1 0; child RH_SHANK -> RR_calf; limit lower=-9.42477796076938 upper=9.42477796076938 effort=80.0 velocity=8.5 -> lower=-2.7227 upper=-0.83776 effort=45.43 velocity=15.70; origin xyz=0 0 0 rpy=0 0 0 -> xyz=0 0 -0.213 rpy=0 0 0; parent RH_KFE_drive -> RR_thigh
- joint imu_joint: axis (none) -> 0 0 0; child imu_link -> imu; origin xyz=-0.25565 0.00255 0.07672 rpy=3.141592653589793 0.0 3.141592653589793 -> xyz=-0.02557 0 0.04232 rpy=0 0 0
