Commit message: update collision sensors

File: tbai_ros_description/urdf/anymal_d_gazebo.urdf.xacro (robot description, xacro)
@@ -186,5 +186,5 @@
     <plugin name="lf_contact_plugin" filename="libContactSensor.so"/>
     <contact>
-        <collision>LF_SHANK_fixed_joint_lump__LF_FOOT_collision_3</collision>
+        <collision>LF_SHANK_fixed_joint_lump__LF_FOOT_collision_sensor_collision_3</collision>
     </contact>
     </sensor>
@@ -194,5 +194,5 @@
     <plugin name="rf_contact_plugin" filename="libContactSensor.so"/>
     <contact>
-        <collision>RF_SHANK_fixed_joint_lump__RF_FOOT_collision_3</collision>
+        <collision>RF_SHANK_fixed_joint_lump__RF_FOOT_collision_sensor_collision_3</collision>
     </contact>
     </sensor>
@@ -202,5 +202,5 @@
     <plugin name="lh_contact_plugin" filename="libContactSensor.so"/>
     <contact>
-        <collision>LH_SHANK_fixed_joint_lump__LH_FOOT_collision_3</collision>
+        <collision>LH_SHANK_fixed_joint_lump__LH_FOOT_collision_sensor_collision_3</collision>
     </contact>
     </sensor>
@@ -210,5 +210,5 @@
     <plugin name="rh_contact_plugin" filename="libContactSensor.so"/>
     <contact>
-        <collision>RH_SHANK_fixed_joint_lump__RH_FOOT_collision_3</collision>
+        <collision>RH_SHANK_fixed_joint_lump__RH_FOOT_collision_sensor_collision_3</collision>
     </contact>
     </sensor>

File: tbai_ros_description/urdf/anymal_d_gazebo_blind.urdf.xacro (robot description, xacro)
@@ -37,5 +37,5 @@
     <plugin name="lf_contact_plugin" filename="/home/kuba/Documents/ros/devel/.private/tbai_ros_gazebo/lib/libContactSensor.so"/>
     <contact>
-        <collision>FL_calf_fixed_joint_lump__LF_FOOT_collision_sensor_collision_3</collision>
+        <collision>LF_SHANK_fixed_joint_lump__LF_FOOT_collision_sensor_collision_3</collision>
     </contact>
     </sensor>
@@ -45,5 +45,5 @@
     <plugin name="rf_contact_plugin" filename="/home/kuba/Documents/ros/devel/.private/tbai_ros_gazebo/lib/libContactSensor.so"/>
     <contact>
-        <collision>FR_calf_fixed_joint_lump__RF_FOOT_collision_sensor_collision_3</collision>
+        <collision>RF_SHANK_fixed_joint_lump__RF_FOOT_collision_sensor_collision_3</collision>
     </contact>
     </sensor>
@@ -53,5 +53,5 @@
     <plugin name="lh_contact_plugin" filename="/home/kuba/Documents/ros/devel/.private/tbai_ros_gazebo/lib/libContactSensor.so"/>
     <contact>
-        <collision>RL_calf_fixed_joint_lump__LH_FOOT_collision_sensor_collision_1</collision>
+        <collision>LH_SHANK_fixed_joint_lump__LH_FOOT_collision_sensor_collision_3</collision>
     </contact>
     </sensor>
@@ -61,5 +61,5 @@
     <plugin name="rh_contact_plugin" filename="/home/kuba/Documents/ros/devel/.private/tbai_ros_gazebo/lib/libContactSensor.so"/>
     <contact>
-        <collision>RR_calf_fixed_joint_lump__RH_FOOT_collision_sensor_collision_1</collision>
+        <collision>RH_SHANK_fixed_joint_lump__RH_FOOT_collision_sensor_collision_3</collision>
     </contact>
     </sensor>

Commit message: small tweaks

File: tbai_ros_description/urdf/anymal_d_gazebo.urdf.xacro (robot description, xacro)
@@ -1,39 +1,39 @@
 <?xml version="1.0"?>
 <robot xmlns:xacro="http://www.ros.org/wiki/xacro" name="anymal_d">
-<!-- Includes -->
-<xacro:include filename="utils.xacro" />
-<!-- Anymal D bare urdf -->
-<xacro:include filename="$(find ocs2_robotic_assets)/resources/anymal_d/urdf/anymal.urdf" />
-<!-- Transmissions LF -->
-<xacro:transmission name="transmission_LF_HAA" joint="LF_HAA" actuator="motor_LF_HAA"/>
-<xacro:transmission name="transmission_LF_HFE" joint="LF_HFE" actuator="motor_LF_HFE"/>
-<xacro:transmission name="transmission_LF_KFE" joint="LF_KFE" actuator="motor_LF_KFE"/>
-<!-- Transmissions LH -->
-<xacro:transmission name="transmission_LH_HAA" joint="LH_HAA" actuator="motor_LH_HAA"/>
-<xacro:transmission name="transmission_LH_HFE" joint="LH_HFE" actuator="motor_LH_HFE"/>
-<xacro:transmission name="transmission_LH_KFE" joint="LH_KFE" actuator="motor_LH_KFE"/>
-<!-- Transmissions RF -->
-<xacro:transmission name="transmission_RF_HAA" joint="RF_HAA" actuator="motor_RF_HAA"/>
-<xacro:transmission name="transmission_RF_HFE" joint="RF_HFE" actuator="motor_RF_HFE"/>
-<xacro:transmission name="transmission_RF_KFE" joint="RF_KFE" actuator="motor_RF_KFE"/>
-<!-- Transmissions RH -->
-<xacro:transmission name="transmission_RH_HAA" joint="RH_HAA" actuator="motor_RH_HAA"/>
-<xacro:transmission name="transmission_RH_HFE" joint="RH_HFE" actuator="motor_RH_HFE"/>
-<xacro:transmission name="transmission_RH_KFE" joint="RH_KFE" actuator="motor_RH_KFE"/>
-<!-- Joint controller -->
-<gazebo>
-  <plugin filename="libgazebo_ros_control.so" name="gazebo_ros_control">
-    <robotSimType>gazebo_ros_control/DefaultRobotHWSim</robotSimType>
-    <robotNamespace>/anymal_d</robotNamespace>
-  </plugin>
-</gazebo>
-<!-- State publisher - enabled or disabled based on the config file -->
-<gazebo>
-  <plugin filename="libStatePublisher.so" name="StatePublisher"/>
-</gazebo>
-<gazebo>
-  <plugin filename="libRobotStatePublisher.so" name="RobotStatePublisher"/>
-</gazebo>
- <joint name="face_front_to_depth_camera_front_camera" type="fixed">
+    <!-- Includes -->
+    <xacro:include filename="utils.xacro" />
+    <!-- Anymal D bare urdf -->
+    <xacro:include filename="$(find ocs2_robotic_assets)/resources/anymal_d/urdf/anymal.urdf" />
+    <!-- Transmissions LF -->
+    <xacro:transmission name="transmission_LF_HAA" joint="LF_HAA" actuator="motor_LF_HAA"/>
+    <xacro:transmission name="transmission_LF_HFE" joint="LF_HFE" actuator="motor_LF_HFE"/>
+    <xacro:transmission name="transmission_LF_KFE" joint="LF_KFE" actuator="motor_LF_KFE"/>
+    <!-- Transmissions LH -->
+    <xacro:transmission name="transmission_LH_HAA" joint="LH_HAA" actuator="motor_LH_HAA"/>
+    <xacro:transmission name="transmission_LH_HFE" joint="LH_HFE" actuator="motor_LH_HFE"/>
+    <xacro:transmission name="transmission_LH_KFE" joint="LH_KFE" actuator="motor_LH_KFE"/>
+    <!-- Transmissions RF -->
+    <xacro:transmission name="transmission_RF_HAA" joint="RF_HAA" actuator="motor_RF_HAA"/>
+    <xacro:transmission name="transmission_RF_HFE" joint="RF_HFE" actuator="motor_RF_HFE"/>
+    <xacro:transmission name="transmission_RF_KFE" joint="RF_KFE" actuator="motor_RF_KFE"/>
+    <!-- Transmissions RH -->
+    <xacro:transmission name="transmission_RH_HAA" joint="RH_HAA" actuator="motor_RH_HAA"/>
+    <xacro:transmission name="transmission_RH_HFE" joint="RH_HFE" actuator="motor_RH_HFE"/>
+    <xacro:transmission name="transmission_RH_KFE" joint="RH_KFE" actuator="motor_RH_KFE"/>
+    <!-- Joint controller -->
+    <gazebo>
+    <plugin filename="libgazebo_ros_control.so" name="gazebo_ros_control">
+        <robotSimType>gazebo_ros_control/DefaultRobotHWSim</robotSimType>
+        <robotNamespace>/anymal_d</robotNamespace>
+    </plugin>
+    </gazebo>
+    <!-- State publisher - enabled or disabled based on the config file -->
+    <gazebo>
+    <plugin filename="libStatePublisher.so" name="StatePublisher"/>
+    </gazebo>
+    <gazebo>
+    <plugin filename="libRobotStatePublisher.so" name="RobotStatePublisher"/>
+    </gazebo>
+    <joint name="face_front_to_depth_camera_front_camera" type="fixed">
         <parent link="face_front"/>
         <child link="depth_camera_front_camera"/>
